Commit message: homer_model string mit elissa3_homer ersetzt

File: urdf/homer.urdf (robot description, URDF)
Before this commit: robot homer, 4 links, 3 joints
Links:
- link base_link: geometry collision mesh filename=package://elissa3_homer/homer_parts/Base_End.stl scale=0.01 0.01 0.01; visual mesh filename=package://elissa3_homer/homer_parts/Base_End.stl scale=0.01 0.01 0.01
- link first_link: geometry collision mesh filename=package://elissa3_homer/homer_parts/Mid.stl scale=0.01 0.01 0.01; visual mesh filename=package://elissa3_homer/homer_parts/Mid.stl scale=0.01 0.01 0.01
- link second_link: geometry collision mesh filename=package://elissa3_homer/homer_parts/Mid.stl scale=0.01 0.01 0.01; visual mesh filename=package://elissa3_homer/homer_parts/Mid.stl scale=0.01 0.01 0.01
